File: Circuits/Teensy max PCB with flip flap/Circuit.brd (EAGLE design)
At the start: 84.3 x 101.3 mm, 50 parts, among them IC1 ULN2003AN, IC2 7805TV, J1 RJ11, J3 POWER_JACK, J4 RJ11, J5 RJ11, J6 POWER_JACK, J7 POWER_JACK, J8 ARDUINO_NANO, J9 POWER_JACK, Q1 IRL540, Q2 IRL540, Q3 IRL540, Q4 IRL540, T1 Z0103MA

Commit message: New circuit
Parts:
- removed C7: 10uF, rcl:E2-5
- removed C9: 10nF, rcl:C050-024X044
- removed J5: RJ11, SparkFun-Connectors:RJ11-6
- removed OK1: MOC3063, optocoupler:DIL06
- removed R6: 390R, rcl:0204/5
- removed R7, R8: 330R, rcl:0204/5
- removed R9: 39R, rcl:0204/5
- removed T1: Z0103MA, triac:TO92-6
- added JP4: COIN CELL, pinhead:1X02
- added L1: 100uH, rcl:6000-XXXX-RC
- C6: value 470uF -> 100uF; device rcl:E3,5-8 -> rcl:E2,5-7
- J2: value (none) -> RJ11; device SparkFun-Connectors:1X01_OFFSET -> SparkFun-Connectors:RJ11-6
- JP2: value HIGH VOLTAGE -> INVERTER OUT
- moved JP1 25.0 mm to (76.2, 74.2)
- moved C6 22.9 mm to (76.2, 68.6), turned to 180 degrees
- moved JP2 14.9 mm to (64.8, 50.8)
- moved J2 1.80 mm to (78.9, 55.5), flipped to the top
Connections:
- removed net N$20: OK1.6, R7.1
- removed net N$21: JP2.1, R7.2, R9.2, T1.A2
- removed net N$22: J5.5, JP2.2
- removed net N$24: C9.1, R9.1
- removed net N$26: J2.1, J5.4
- net +12V: now also L1.1; no longer JP1.1
- net +7V: now also J2.5; no longer C6.+, C7.+, J5.1
- net GND: now also J2.6, JP4.1; no longer C6.-, C7.-, J5.3, R6.1
- net N$12: now also C6.+, JP1.1, L1.2; no longer OK1.2, R6.2
- net N$13: now also J2.1, JP2.1; no longer J8.J1.14, OK1.1
- net N$14: now also J2.2, JP2.2; no longer OK1.4, R8.1, T1.G
- net N$15: now also JP4.2, U$1.VBAT\; no longer C9.2, J5.6, R8.2, T1.A1
- net N$3: now also C6.-
- net SERVO: now also J2.4; no longer J5.2
Routing:
- net N$15: track 62.7 -> 3.54 mm
- net +12V: track 329.8 -> 359.6 mm
- net N$21: track 23.5 -> 0.00 mm
- net +7V: track 138.7 -> 161.9 mm
- net GND: track 593.6 -> 573.0 mm
- net N$3: track 20.1 -> 39.4 mm
- net SERVO: track 48.1 -> 30.8 mm
- net N$22: track 13.6 -> 0.00 mm
- net N$12: track 11.2 -> 19.3 mm
- net N$20: track 6.62 -> 0.00 mm
- net N$26: track 5.21 -> 0.00 mm
- net N$14: track 10.8 -> 12.8 mm
- net N$24: track 1.59 -> 0.00 mm
