File: Circuits/Teensy max PCB with flip flap/Circuit.sch (EAGLE design)
At the start: 50 parts, among them IC1 ULN2003AN, IC2 7805TV, J1 RJ11, J3 POWER_JACK, J4 RJ11, J5 RJ11, J6 POWER_JACK, J7 POWER_JACK, J8 ARDUINO_NANO, J9 POWER_JACK, Q1 IRL540, Q2 IRL540, Q3 IRL540, Q4 IRL540, T1 Z0103MA

Commit message: New circuit
Parts:
- removed C7: 10uF, rcl:CPOL-EUE2-5
- removed C9: 10nF, rcl:C-EU050-024X044
- removed J5: RJ11, SparkFun-Connectors:RJ11-6
- removed OK1: MOC3063, optocoupler:MOC3043M
- removed R6: 390R, rcl:R-EU_0204/5
- removed R7, R8: 330R, rcl:R-EU_0204/5
- removed R9: 39R, rcl:R-EU_0204/5
- removed T1: Z0103MA, triac:TICP206
- added JP4: COIN CELL, pinhead:PINHD-1X2
- added L1: 100uH, rcl:L-US6000-XXX-RC
- C6: value 470uF -> 100uF; device rcl:CPOL-EUE3.5-8 -> rcl:CPOL-USE2.5-7
- J2: value (none) -> RJ11; device SparkFun-Connectors:CONN_01OFFSET -> SparkFun-Connectors:RJ11-6
- JP2: value HIGH VOLTAGE -> INVERTER OUT
Connections:
- removed net N$20: OK1.A2, R7.1
- removed net N$21: JP2.1, R7.2, R9.2, T1.A2
- removed net N$22: J5.5, JP2.2
- removed net N$24: C9.1, R9.1
- removed net N$26: J2.1, J5.4
- net +12V: now also L1.1; no longer JP1.1
- net +7V: now also J2.5; no longer C6.+, C7.+, J5.1
- net GND: now also J2.6, JP4.1; no longer C6.-, C7.-, J5.3, R6.1
- net N$12: now also C6.+, JP1.1, L1.2; no longer OK1.C, R6.2
- net N$13: now also J2.1, JP2.1; no longer J8.D11/MOSI, OK1.A
- net N$14: now also J2.2, JP2.2; no longer OK1.A1, R8.1, T1.G
- net N$15: now also JP4.2, U$1.VBAT; no longer C9.2, J5.6, R8.2, T1.A1
- net N$3: now also C6.-
- net SERVO: now also J2.4; no longer J5.2
Other:
- note added: "Buck converter for EL panel"
- moved on the sheet: C1, C2, C3, C4, C5, C6, C8, D1, D2, D3, D4, DRV1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
